Commit message: fixed global camera calibratoin

File: Motion/data/robots/Bubonic_no_camera.urdf (robot description, URDF)
Before this commit: robot Lowpoly_anthrax_URDF, 17 links, 16 joints
Links:
- link base_link: geometry collision mesh filename=Anthrax_lowpoly/base_link_Adjusted.STL; visual mesh filename=Anthrax_lowpoly/base_link_Adjusted.STL
- link left_EE_link: geometry collision mesh filename=Anthrax_lowpoly/left_EE_link.STL; visual mesh filename=Anthrax_lowpoly/left_EE_link.STL
- link left_base_link: geometry collision mesh filename=Anthrax_lowpoly/left_base_link.STL; visual mesh filename=Anthrax_lowpoly/left_base_link.STL
- link left_forearm_link: geometry collision mesh filename=Anthrax_lowpoly/left_forearm_link.STL; visual mesh filename=Anthrax_lowpoly/left_forearm_link.STL
- link left_shoulder_link: geometry collision mesh filename=Anthrax_lowpoly/left_shoulder_link.STL; visual mesh filename=Anthrax_lowpoly/left_shoulder_link.STL
- link left_upperarm_link: geometry collision mesh filename=Anthrax_lowpoly/left_upperarm_link.STL; visual mesh filename=Anthrax_lowpoly/left_upperarm_link.STL
- link left_wrist1_link: geometry collision mesh filename=Anthrax_lowpoly/left_wrist1_link.STL; visual mesh filename=Anthrax_lowpoly/left_wrist1_link.STL
- link left_wrist2_link: geometry collision mesh filename=Anthrax_lowpoly/left_wrist2_link.STL; visual mesh filename=Anthrax_lowpoly/left_wrist2_link.STL
- link left_wrist3_link: geometry collision mesh filename=Anthrax_lowpoly/left_wrist3_link_Adjusted.STL; visual mesh filename=Anthrax_lowpoly/left_wrist3_link_Adjusted.STL
- link right_EE_link: geometry collision mesh filename=Anthrax_lowpoly/right_EE_link.STL; visual mesh filename=Anthrax_lowpoly/right_EE_link.STL
- link right_base_link: geometry collision mesh filename=Anthrax_lowpoly/right_base_link.STL; visual mesh filename=Anthrax_lowpoly/right_base_link.STL
- link right_forearm_link: geometry collision mesh filename=Anthrax_lowpoly/right_forearm_link.STL; visual mesh filename=Anthrax_lowpoly/right_forearm_link.STL
- link right_shoulder_link: geometry collision mesh filename=Anthrax_lowpoly/right_shoulder_link.STL; visual mesh filename=Anthrax_lowpoly/right_shoulder_link.STL
- link right_upperarm_link: geometry collision mesh filename=Anthrax_lowpoly/right_upperarm_link.STL; visual mesh filename=Anthrax_lowpoly/right_upperarm_link.STL
- link right_wrist1_link: geometry collision mesh filename=Anthrax_lowpoly/right_wrist1_link.STL; visual mesh filename=Anthrax_lowpoly/right_wrist1_link.STL
- link right_wrist2_link: geometry collision mesh filename=Anthrax_lowpoly/right_wrist2_link.STL; visual mesh filename=Anthrax_lowpoly/right_wrist2_link.STL
- link right_wrist3_link: geometry collision mesh filename=Anthrax_lowpoly/right_wrist3_link_Adjusted.STL; visual mesh filename=Anthrax_lowpoly/right_wrist3_link_Adjusted.STL
Joints:
- joint base_left_base: origin xyz=-0.105005 -0.717077 0.563484 rpy=0.631490 0.478004 -2.040709 -> xyz=0.019917 0.181 1.2870299 rpy=0.615191 0.523936 2.525974
- joint base_right_base: origin xyz=0.243036 -0.661803 0.551280 rpy=-0.590603 0.476972 -0.874202 -> xyz=0.020083 -0.181 1.2870297 rpy=-0.615791 0.523201 -2.526274

File: Motion/data/robots/Bubonic_uncalibrated.urdf (robot description, URDF)
Before this commit: robot Lowpoly_anthrax_URDF, 17 links, 16 joints
Links:
- link base_link: geometry collision mesh filename=Bubonic_zherong/base_link_Adjusted.STL; visual mesh filename=Bubonic_zherong/base_link_Adjusted.STL
Joints:
- joint base_left_base: origin xyz=-0.105005 -0.717077 0.563484 rpy=0.631490 0.478004 -2.040709 -> xyz=0.019917 0.180606 1.286799 rpy=0.615191 0.523936 2.525974
- joint base_right_base: origin xyz=0.243036 -0.661803 0.551280 rpy=-0.590603 0.476972 -0.874202 -> xyz=0.020083 -0.180588 1.286797 rpy=-0.615791 0.523201 -2.526274

Commit message: Testing

File: Motion/data/robots/Bubonic_no_camera.urdf (robot description, URDF)
Before this commit: robot Lowpoly_anthrax_URDF, 17 links, 16 joints
Links:
- link left_wrist3_link: geometry collision mesh filename=Anthrax_lowpoly/left_wrist3_link.STL; visual mesh filename=Anthrax_lowpoly/left_wrist3_link.STL
- link right_wrist3_link: geometry collision mesh filename=Anthrax_lowpoly/right_wrist3_link.STL; visual mesh filename=Anthrax_lowpoly/right_wrist3_link.STL
