Commit message: Fixed robotiq model, drivers work and can now be simulated properly

File: Motion/data/robots/robotiq_140.urdf (robot description, URDF)
Before this commit: robot robotiq_140, 11 links, 10 joints
Links:
- added link world
- link base_link: mass 163.626380453613 -> 0.86247164
Joints:
- added joint freeze_base_joint: type fixed, parent world, child base_link
