Commit message: added grippers to Cholera

File: Motion/data/robots/Cholera.urdf (robot description, URDF)
Before this commit: robot Cholera, 21 links, 20 joints
Links:
- added link sucker_link, mass 2.5E-05; collision mesh filename=other/Epick_assembly.STL; visual mesh filename=other/Epick_assembly.STL
Joints:
- added joint sucker_joint: type fixed, parent right_tool_link, child sucker_link, origin xyz=0 0 0 rpy=0 1.5708 0, axis 0 0 0

Commit message: fix one bug in Cholera

File: Motion/data/robots/Cholera.urdf (robot description, URDF)
Before this commit: robot Cholera, 22 links, 21 joints
Joints:
- joint right_wrist1_wrist2: origin xyz=0 0.0462999999999996 0.0589 rpy=1.5707963267949 1.5707963267949 -3.14159265358979 -> xyz=0 0.0462999999999996 0.0589 rpy=1.5707963267949 0 -3.14159265358979

Commit message: Tuning collision margin

File: Motion/data/robots/Cholera.urdf (robot description, URDF)
Before this commit: robot Cholera, 22 links, 21 joints
Joints:
- joint sucker_joint: origin xyz=0 0 0 rpy=0 1.5708 0 -> xyz=0 0 0 rpy=1.5708 0 1.5708

Commit message: updated calibrated cholera

File: Motion/data/robots/Cholera.urdf (robot description, URDF)
Before this commit: robot Cholera, 22 links, 21 joints
Links:
- link base_link: geometry collision mesh filename=Cholera_calibrated/base_link.STL; visual mesh filename=Cholera_calibrated/base_link.STL
- link left_wrist2_link: geometry collision mesh filename=Cholera_calibrated/left_wrist2_link.STL; visual mesh filename=Cholera_calibrated/left_wrist2_link.STL
- link right_wrist2_link: geometry collision mesh filename=Cholera_calibrated/right_wrist2_link.STL; visual mesh filename=Cholera/right_wrist2_link.STL
Joints:
- joint base_left_base: origin xyz=0.0199169066321389 0.184218468750741 1.1474483982822 rpy=2.52611294491941 0.523598775598306 -2.52566187507049 -> xyz=0.0012562098034254498 0.1932543267616293 1.2569858725693364 rpy=2.5100806626787446 0.4846408201341714 3.7518758665533896
- joint base_right_base: origin xyz=0.0200830892985796 -0.184200425957397 1.1474483982822 rpy=-2.5261129449194 0.523598775598298 2.52656401476832 -> xyz=0.0010313332699722 -0.19888109142120516 1.2534172095913139 rpy=3.7445696646064053 0.5074053284196887 2.517032028984335

Commit message: 0124 calibration tests

File: Motion/data/robots/Cholera.urdf (robot description, URDF)
Before this commit: robot Cholera, 22 links, 21 joints
Joints:
- joint base_left_base: origin xyz=0.0012562098034254498 0.1932543267616293 1.2569858725693364 rpy=2.5100806626787446 0.4846408201341714 3.7518758665533896 -> xyz=-0.02952606997846065 0.22582869698830485 1.2367235895316024 rpy=2.5624285536623925 0.4879984171093927 3.739748420340416

Commit message: 0127 calibration of the left camera

File: Motion/data/robots/Cholera.urdf (robot description, URDF)
Before this commit: robot Cholera, 22 links, 21 joints
Joints:
- joint base_left_base: origin xyz=-0.02952606997846065 0.22582869698830485 1.2367235895316024 rpy=2.5624285536623925 0.4879984171093927 3.739748420340416 -> xyz=-0.01340967183126901, 0.18598624997360852, 1.2618577587021373 rpy=2.5119266093029307 0.5226624603087614 3.721560774297633
